File: hardware/psu/psu.kicad_sch (KiCad schematic)
At the start: 46 parts, among them J1 Conn_02x08_Odd_Even, J2 Conn_02x02_Odd_Even, J3 USB_C_Receptacle_USB2.0_14P, J4 USB_A, Q1 DMP3056LSS, SW1 SW_SPDT, U1 REC30K-2412DZ, U2 CH224A, U3 AP63301WU

Commit message: Version 1.1 board. Measurements complete, updated power on switch design, refined in-rush limiting
Parts:
- removed SW1: SW_SPDT, Switches:SW_300SP1J1BLKM6QE, symbol Switch:SW_SPDT
- added C19: 100n, Capacitor_SMD:C_0805_2012Metric_Pad1.18x1.45mm_HandSolder, symbol Device:C
- added C20: 1u, Capacitor_SMD:C_0805_2012Metric_Pad1.18x1.45mm_HandSolder, symbol Device:C
- added Q2: 2N7002, Package_TO_SOT_SMD:SOT-23, symbol Transistor_FET:2N7002
- added R10: 100k, Resistor_SMD:R_0805_2012Metric_Pad1.20x1.40mm_HandSolder, symbol Device:R_US
- added R11: 47k, Resistor_SMD:R_0805_2012Metric_Pad1.20x1.40mm_HandSolder, symbol Device:R_US
- added R12, R13: 15k, Resistor_SMD:R_0805_2012Metric_Pad1.20x1.40mm_HandSolder, symbol Device:R_US
- added R14: 220, Resistor_SMD:R_0805_2012Metric_Pad1.20x1.40mm_HandSolder, symbol Device:R_US
- added SW2: SW_Slide_DPDT, Switches:SW_DPDT_LC2255EENP, symbol Modular_Switches:SW_Slide_DPDT_Shielded
- C12: value 100n -> 1u
- D2: footprint LED_SMD:LED_1206_3216Metric_Pad1.42x1.75mm_HandSolder -> LED_SMD:LED_0805_2012Metric_Pad1.15x1.40mm_HandSolder
- R1: value 4k7 -> 2k2
- R2, R3: footprint Resistor_SMD:R_2512_6332Metric_Pad1.40x3.35mm_HandSolder -> Resistor_SMD:R_1206_3216Metric_Pad1.30x1.75mm_HandSolder
- R7: value 1k0 -> 4k7
Connections:
- net VUSB_C is gone; now on net VDC_SYS: C13.1, Q1.5 (D), Q1.6 (D), Q1.7 (D), Q1.8 (D)
- net +12V: now also J2.2 (Pin_2), R10.1; no longer J2.3 (Pin_3)
- net +5V: now also D1.2 (A), J2.3 (Pin_3); no longer J2.4 (Pin_4)
- net -12V: now also J2.4 (Pin_4); no longer J2.1 (Pin_1)
- net GND: now also J2.1 (Pin_1), C19.1, C20.1, Q2.2 (S), R11.2, R13.2, SW2.1 (A), SW2.4 (A), SW2.SH (A); no longer J2.2 (Pin_2)
- net VDC_SYS: now also R12.1; no longer D1.2 (A), U3.2 (EN)
- net at U1.3 (CTRL): now also Q2.3 (D)
- new net: C20.2, R14.2
- new net: C19.2, R10.2, R11.1, U3.2 (EN)
- new net DC_PWR_ON: Q2.1 (G), R12.2, R13.1, R14.1, SW2.2 (B), SW2.5 (B)
Other:
- note added: "1W"
- moved on the sheet: C1, C14, C15, C16, C17, C18, C2, C3, C4, C5, C6, C7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
