File: hardware/psu/psu.kicad_sch (KiCad schematic)
At the start: 54 parts, among them J1 Conn_02x08_Odd_Even, J2 Conn_02x02_Odd_Even, J3 USB_C_Receptacle_USB2.0_14P, J4 USB_A, Q1 DMP3056LSS, Q2 2N7002, SW2 SW_Slide_DPDT, U1 REC30K-2412DZ, U2 CH224A, U3 AP63301WU

Commit message: Fixed ref for SW1, updated BOM for v1.1
Parts:
- renumbered SW2 to SW1
Changed lines of the file:
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@@
 		(dnp no)
 		(fields_autoplaced yes)
-		(property "Reference" "SW2"
+		(property "Reference" "SW1"
 			(at 83.82 153.67 0)
 			(effects
@@
 			(project "psu"
 				(path "/dcf32edd-aaf4-447c-a68f-dcd4630a380b"
-					(reference "SW2")
+					(reference "SW1")
 					(unit 1)
 				)

Commit message: Fix power on behavior with delay C to ground on REC30K CTRL, tick board rev to 1.2
Parts:
- added C21: 3u3, Capacitor_SMD:C_0805_2012Metric_Pad1.18x1.45mm_HandSolder, symbol Device:C
- added R15: 220, Resistor_SMD:R_0805_2012Metric_Pad1.20x1.40mm_HandSolder, symbol Device:R_US
Connections:
- net GND: now also C21.1
- net at Q2.3 (D), U1.3 (CTRL): now also R15.1
- new net: C21.2, R15.2

Commit message: Rev 1.3 board with ESD protection and current protection for the USB A output (not fabricated yet)
Parts:
- added C22: 220u, Capacitors_Custom:CAP_UCD_6P3X7P7_NCH, symbol Device:C_Polarized_US
- added C23, C24: 100n, Capacitor_SMD:C_0805_2012Metric_Pad1.18x1.45mm_HandSolder, symbol Device:C
- added D4, D5, D6: TSD05D, Diode_SMD:D_SOD-323_HandSoldering, symbol Device:D_Zener
- added D7, D8: TSD03D, Diode_SMD:D_SOD-323_HandSoldering, symbol Device:D_Zener
- added D9: TSD18D, Diode_SMD:D_SOD-323_HandSoldering, symbol Device:D_Zener
- added R16: 22k, Resistor_SMD:R_0805_2012Metric_Pad1.20x1.40mm_HandSolder, symbol Device:R_US
- added R17: 100k, Resistor_SMD:R_0805_2012Metric_Pad1.20x1.40mm_HandSolder, symbol Device:R_US
- added U4: TPS2553D, Package_TO_SOT_SMD:SOT-23-6_Handsoldering, symbol TPS2553:TPS2553DBVR-1
Connections:
- net +5V: now also C23.2, R17.1, U4.1 (IN); no longer J4.1 (VBUS)
- net CC1: now also D5.1 (K)
- net CC2: now also D6.1 (K)
- net GND: now also C22.2, C23.1, C24.1, D4.2 (A), D5.2 (A), D6.2 (A), D7.2 (A), D8.2 (A), D9.2 (A), R16.2, U4.2 (GND)
- net VBUS_IN: now also D9.1 (K)
- net at J3.A6 (D+), J3.B6 (D+), U2.4 (DP): now also D8.1 (K)
- net at J3.A7 (D-), J3.B7 (D-), U2.5 (DM): now also D7.1 (K)
- new net: C24.2, R17.2, U4.3 (EN), U4.4 (FAULT_N)
- new net: R16.1, U4.5 (ILIM)
- new net VBUS_USB_A: C22.1, D4.1 (K), J4.1 (VBUS), U4.6 (OUT)
Other:
- note added: "R_ILM | I_OS(nom) ------|----------- 22k | 1169mA 47k | 556mA"
- moved on the sheet: C1, C10, C14, C15, C16, C17, C18, C19, C2, C20, C21, C3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
