File: hardware/psu/psu.kicad_pcb (KiCad board)
At the start: 4 copper layers, 42 x 100 mm, 54 parts, among them J1 Conn_02x08_Odd_Even, J2 Conn_02x02_Odd_Even, J3 USB_C_Receptacle_USB2.0_14P, J4 USB_A, Q1 DMP3056LSS, Q2 2N7002, SW2 SW_Slide_DPDT, U1 REC30K-2412DZ, U2 CH224A, U3 AP63301WU

Commit message: Fix power on behavior with delay C to ground on REC30K CTRL, tick board rev to 1.2
Parts:
- added C21: 3u3, Capacitor_SMD:C_0805_2012Metric_Pad1.18x1.45mm_HandSolder, F.Cu at (118.0, 80.5)
- added R15: 220, Resistor_SMD:R_0805_2012Metric_Pad1.20x1.40mm_HandSolder, F.Cu at (113.9, 80.5)
- moved C20 0.40 mm to (118.0, 78.1)
- moved Q2 0.40 mm to (109.8, 79.0)
- moved R12 0.40 mm to (113.9, 75.8)
- moved R13 0.40 mm to (109.8, 75.8)
- moved R14 0.40 mm to (113.9, 78.1)
- renumbered SW2 to SW1
Routing:
- net Net-(Q2-D): track 18.6 -> 22.3 mm
- net Net-(C21-Pad2): track 0.00 -> 2.06 mm
- net GND: track 18.0 -> 19.1 mm, vias 68 -> 69

Commit message: Rev 1.3 board with ESD protection and current protection for the USB A output (not fabricated yet)
Parts:
- added C22: 220u, Capacitors_Custom:CAP_UCD_6P3X7P7_NCH, F.Cu at (116.3, 69.9)
- added C23: 100n, Capacitor_SMD:C_0805_2012Metric_Pad1.18x1.45mm_HandSolder, F.Cu at (121.5, 67.3)
- added C24: 100n, Capacitor_SMD:C_0805_2012Metric_Pad1.18x1.45mm_HandSolder, F.Cu at (120.5, 60.6)
- added D4: TSD05D, Diode_SMD:D_SOD-323_HandSoldering, F.Cu at (113.5, 61.7)
- added D5: TSD05D, Diode_SMD:D_SOD-323_HandSoldering, F.Cu at (116.8, 132.5)
- added D6: TSD05D, Diode_SMD:D_SOD-323_HandSoldering, F.Cu at (114.1, 140.6)
- added D7: TSD03D, Diode_SMD:D_SOD-323_HandSoldering, F.Cu at (114.1, 146.1)
- added D8: TSD03D, Diode_SMD:D_SOD-323_HandSoldering, F.Cu at (114.1, 143.3)
- added D9: TSD18D, Diode_SMD:D_SOD-323_HandSoldering, F.Cu at (111.7, 130.8)
- added R16: 22k, Resistor_SMD:R_0805_2012Metric_Pad1.20x1.40mm_HandSolder, F.Cu at (116.5, 60.7)
- added R17: 100k, Resistor_SMD:R_0805_2012Metric_Pad1.20x1.40mm_HandSolder, F.Cu at (121.5, 63.5)
- added U4: TPS2553D, Package_TO_SOT_SMD:SOT-23-6_Handsoldering, F.Cu at (118.0, 63.5)
- moved C18 13.5 mm to (132.5, 61.1), turned to 0 degrees
- moved C17 11.6 mm to (132.5, 58.7), turned to 0 degrees
- moved C10 8.36 mm to (106.9, 130.8), turned to 180 degrees
- moved C11 5.80 mm to (120.2, 142.3)
- moved C12 5.15 mm to (119.8, 139.4)
- moved D3 5.15 mm to (124.2, 139.8)
- moved R5 5.15 mm to (127.7, 144.2)
- moved R7 5.15 mm to (126.5, 139.4)
- moved U2 5.15 mm to (122.4, 146.4)
- moved R6 5.15 mm to (121.8, 139.4)
- moved Q1 1.60 mm to (109.5, 126.0)
- moved C13 1.55 mm to (113.4, 127.5)
- moved R10 1.48 mm to (131.9, 56.1), turned to 180 degrees
- moved R4 1.00 mm to (106.2, 140.5)
- moved C1 0.89 mm to (102.1, 121.6)
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Connections:
- net DC_PWR_ON renamed /DC_PWR_ON
- J4 pad 1: +5V -> /VBUS_USB_A
Routing:
- net GND: track 19.1 -> 30.9 mm, vias 69 -> 92
- net /CC1: track 30.0 -> 38.5 mm
- net Net-(U4-EN): track 0.00 -> 6.95 mm
- net +5V: track 109.9 -> 116.8 mm
- net +12V: track 64.8 -> 69.7 mm
- net Net-(D8-K): track 15.8 -> 20.1 mm, vias 1 -> 0
- net Net-(U4-ILIM): track 0.00 -> 4.11 mm
- net /CC2: track 22.3 -> 26.3 mm, vias 1 -> 2
- net Net-(D3-A): track 18.5 -> 22.1 mm
- net Net-(U3-EN): track 26.0 -> 23.1 mm
- net Net-(D7-K): track 34.9 -> 37.5 mm, vias 2 -> 1
- net VBUS_IN: track 42.7 -> 40.6 mm
- net Net-(D2-K): track 2.77 -> 1.88 mm
- added copper zone on F.Cu, net /VBUS_USB_A
Other:
- board text added: "idyllm CC BY-SA 4.0 v1.3.20261002"
- board text removed: "idyllm CC BY-SA 4.0 v1.1.20260626"
